File: mainboard/mainboard.kicad_pcb (KiCad board)
At the start: 2 copper layers, 70 x 70 mm, 31 parts, among them J1 Barrel_Jack 2.1mm / 2.5A, J2 Screw_Terminal_01x05, J3 Screw_Terminal_01x04, J4 Conn_02x04_Odd_Even, Q1 IRF3708, Q2 IRF3708, Q3 IRF3708, U1 VR10S05, U2 ATmega328P-P, Y1 16Mhz, 20pF

Commit message: added fuse, modified trace widths and added fabrication files
Parts:
- added F1: 3.5A, Resistor_SMD:R_1206_3216Metric, F.Cu at (122.2, 66.2)
Connections:
- J1 pad 1: +12V -> Net-(F1-Pad1)
Routing:
- net Net-(F1-Pad1): track 0.00 -> 27.1 mm, vias 0 -> 1

Commit message: minor changes
Changed lines of the file:
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@@
   (segment (start 163.86 83.16) (end 166.08 83.16) (width 0.2) (layer "F.Cu") (net 35))
   (segment (start 160.03 66.01) (end 160.03 79.33) (width 0.2) (layer "F.Cu") (net 35))
-  (segment (start 122.2 64.7375) (end 122.2 63) (width 2) (layer "F.Cu") (net 36))
+  (segment (start 122.2 64.7375) (end 122.2 63) (width 3) (layer "F.Cu") (net 36))
   (via (at 122.2 63) (size 1.4) (drill 1) (layers "F.Cu" "B.Cu") (net 36))
-  (segment (start 133 74.7) (end 129.2 74.7) (width 2) (layer "B.Cu") (net 36))
-  (segment (start 130.1 63) (end 133.7 66.6) (width 2) (layer "B.Cu") (net 36))
-  (segment (start 129.2 74.7) (end 129.1 74.6) (width 2) (layer "B.Cu") (net 36))
-  (segment (start 133.7 66.6) (end 133.7 74) (width 2) (layer "B.Cu") (net 36))
-  (segment (start 122.2 63) (end 130.1 63) (width 2) (layer "B.Cu") (net 36))
-  (segment (start 133.7 74) (end 133 74.7) (width 2) (layer "B.Cu") (net 36))
+  (segment (start 133 74.7) (end 129.2 74.7) (width 3) (layer "B.Cu") (net 36))
+  (segment (start 130.1 63) (end 133.7 66.6) (width 3) (layer "B.Cu") (net 36))
+  (segment (start 129.2 74.7) (end 129.1 74.6) (width 3) (layer "B.Cu") (net 36))
+  (segment (start 133.7 66.6) (end 133.7 74) (width 3) (layer "B.Cu") (net 36))
+  (segment (start 122.2 63) (end 130.1 63) (width 3) (layer "B.Cu") (net 36))
+  (segment (start 133.7 74) (end 133 74.7) (width 3) (layer "B.Cu") (net 36))
   (zone (net 30) (net_name "+12V") (layer "F.Cu") (hatch edge 0.5)
     (priority 3)

Commit message: generated new fabrication files
Parts:
- R1: value 500 -> 500 / 1/4W
- R2: value 150 -> 150 / 1/10W
Changed lines of the file:
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@@
       (drillshape 0)
       (scaleselection 1)
-      (outputdirectory "/home/maximilian/Desktop/fabrication-files/")
+      (outputdirectory "/home/maximilian/Dokumente/Rücklicht Projekt/LightControl/mainboard/fabrication-files/")
     )
   )
@@
         (effects (font (size 1 1) (thickness 0.15)))
     )
-    (fp_text value "500" (at 0 1.43) (layer "F.Fab")
+    (fp_text value "500 / 1/4W" (at 0 1.43) (layer "F.Fab")
         (effects (font (size 1 1) (thickness 0.15)))
     )
@@
         (effects (font (size 1 1) (thickness 0.15)))
     )
-    (fp_text value "150" (at 0 1.43) (layer "F.Fab")
-        (effects (font (size 1 1) (thickness 0.15)))
-    )
+    (fp_text value "150 / 1/10W" (at 0 1.43) (layer "F.Fab")
+        (effects (font (size 1 1) (thickness 0.15)))
+    )
