File: remote/remote.kicad_pcb (KiCad board)
At the start: 2 copper layers, 30 x 58 mm, 11 parts, among them J4 Screw_Terminal_01x05

Commit message: minor changes
Parts:
- moved H4 1.62 mm to (152.7, 102.4)
- moved H3 1.11 mm to (130.7, 102.4)
- moved H1 0.39 mm to (130.7, 54.4)
- moved H2 0.30 mm to (152.8, 54.4)
Changed lines of the file:
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@@
   (net 5 "IND_BTN")
   (footprint "MountingHole:MountingHole_3.2mm_M3_DIN965_Pad" (layer "F.Cu")
-    (at 130.3 54.3)
+    (at 130.675 54.4)
     (descr "Mounting Hole 3.2mm, M3, DIN965")
     (tags "mounting hole 3.2mm m3 din965")
@@
     (property "Sheetname" "")
     (attr through_hole)
-    (fp_text reference "J1" (at 0 -0.5 unlocked) (layer "F.SilkS")
+    (fp_text reference "J1" (at 9.325 -6 unlocked) (layer "F.SilkS")
         (effects (font (size 1 1) (thickness 0.1)))
     )
@@
     (property "Sheetname" "")
     (attr through_hole)
-    (fp_text reference "J2" (at 0 -0.5 unlocked) (layer "F.SilkS")
+    (fp_text reference "J2" (at 9.425 -5.5 unlocked) (layer "F.SilkS")
         (effects (font (size 1 1) (thickness 0.1)))
     )
@@
   )
   (footprint "MountingHole:MountingHole_3.2mm_M3_DIN965_Pad" (layer "F.Cu")
-    (at 130.2 103.4)
+    (at 130.675 102.4)
     (descr "Mounting Hole 3.2mm, M3, DIN965")
     (tags "mounting hole 3.2mm m3 din965")
@@
   )
   (footprint "MountingHole:MountingHole_3.2mm_M3_DIN965_Pad" (layer "F.Cu")
-    (at 153.3 103.9)
+    (at 152.675 102.4)
     (descr "Mounting Hole 3.2mm, M3, DIN965")
     (tags "mounting hole 3.2mm m3 din965")
@@
   )
   (footprint "MountingHole:MountingHole_3.2mm_M3_DIN965_Pad" (layer "F.Cu")
-    (at 152.8 54.1)
+    (at 152.8 54.4)
     (descr "Mounting Hole 3.2mm, M3, DIN965")
     (tags "mounting hole 3.2mm m3 din965")
@@
     (property "Sheetname" "")
     (attr through_hole)
-    (fp_text reference "J3" (at 0 -0.5 unlocked) (layer "F.SilkS")
+    (fp_text reference "J3" (at 9.325 -5.4 unlocked) (layer "F.SilkS")
         (effects (font (size 1 1) (thickness 0.1)))
     )
@@
       )
     )
+  )
+  (zone (net 0) (net_name "") (layer "F.Cu") (hatch edge 0.5)
+    (connect_pads (clearance 0))
+    (min_thickness 0.25) (filled_areas_thickness no)
+    (keepout (tracks allowed) (vias allowed) (pads allowed) (copperpour not_allowed) (footprints allowed))
+    (fill (thermal_gap 0.5) (thermal_bridge_width 0.5))
+    (polygon
+      (pts
+        (xy 143.8 51.3)
+        (xy 146.2 51.3)
+        (xy 146.2 52.2)
+        (xy 143.8 52.2)
+      )
+    )

Commit message: generated new fabrication files
Parts:
- J1, J2, J3: value ~ -> 12mm non-resetting button
Other:
- board text added: "JLCJLCJLCJLC"
- board text added: "LightControl Remote V1.0 03/2023 M. Stucke"
Changed lines of the file:
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@@
   )
   (paper "A4")
+  (title_block
+    (title "LightControl Remote")
+    (date "2023-03-27")
+    (rev "1.0")
+    (company "Maximilian Stucke")
+  )
   (layers
     (0 "F.Cu" signal)
@@
       (outputformat 1)
       (mirror false)
-      (drillshape 1)
+      (drillshape 0)
       (scaleselection 1)
-      (outputdirectory "")
+      (outputdirectory "/home/maximilian/Dokumente/Rücklicht Projekt/LightControl/remote/fabrication files/")
     )
   )
@@
     (descr "Mounting Hole 3.2mm, M3, DIN965")
     (tags "mounting hole 3.2mm m3 din965")
-    (property "Sheetfile" "remote-project.kicad_sch")
+    (property "Sheetfile" "remote.kicad_sch")
     (property "Sheetname" "")
     (property "ki_description" "Mounting Hole with connection")
@@
     (descr "Resistor SMD 0603 (1608 Metric), square (rectangular) end terminal, IPC_7351 nominal, (Body size source: IPC-SM-782 page 72, https://www.pcb-3d.com/wordpress/wp-content/uploads/ipc-sm-782a_amendment_1_and_2.pdf), generated with kicad-footprint-generator")
     (tags "resistor")
-    (property "Sheetfile" "remote-project.kicad_sch")
+    (property "Sheetfile" "remote.kicad_sch")
     (property "Sheetname" "")
     (property "ki_description" "Resistor, small symbol")
@@
     (descr "Resistor SMD 0603 (1608 Metric), square (rectangular) end terminal, IPC_7351 nominal, (Body size source: IPC-SM-782 page 72, https://www.pcb-3d.com/wordpress/wp-content/uploads/ipc-sm-782a_amendment_1_and_2.pdf), generated with kicad-footprint-generator")
     (tags "resistor")
-    (property "Sheetfile" "remote-project.kicad_sch")
+    (property "Sheetfile" "remote.kicad_sch")
     (property "Sheetname" "")
     (property "ki_description" "Resistor, small symbol")
@@
     (descr "Resistor SMD 0603 (1608 Metric), square (rectangular) end terminal, IPC_7351 nominal, (Body size source: IPC-SM-782 page 72, https://www.pcb-3d.com/wordpress/wp-content/uploads/ipc-sm-782a_amendment_1_and_2.pdf), generated with kicad-footprint-generator")
     (tags "resistor")
-    (property "Sheetfile" "remote-project.kicad_sch")
+    (property "Sheetfile" "remote.kicad_sch")
     (property "Sheetname" "")
     (property "ki_description" "Resistor, small symbol")
@@
   (footprint "Button_Switch:5V_LED_BTN" (layer "F.Cu")
     (at 141.675 68.9)
-    (property "Sheetfile" "remote-project.kicad_sch")
+    (property "Sheetfile" "remote.kicad_sch")
     (property "Sheetname" "")
     (attr through_hole)
@@
         (effects (font (size 1 1) (thickness 0.1)))
     )
-    (fp_text value "~" (at 0 1 unlocked) (layer "F.Fab")
+    (fp_text value "12mm non-resetting button" (at 0 1 unlocked) (layer "F.Fab")
         (effects (font (size 1 1) (thickness 0.15)))
     )
@@
     (descr "Terminal Block TE 282834-5, 5 pins, pitch 2.54mm, size 13.16x6.5mm^2, drill diamater 1.1mm, pad diameter 2.1mm, see http://www.te.com/commerce/DocumentDelivery/DDEController?Action=showdoc&DocId=Customer+Drawing%7F282834%7FC1%7Fpdf%7FEnglish%7FENG_CD_282834_C1.pdf, script-generated using https://github.com/pointhi/kicad-footprint-generator/scripts/TerminalBlock_TE-Connectivity")
     (tags "THT Terminal Block TE 282834-5 pitch 2.54mm size 13.16x6.5mm^2 drill 1.1mm pad 2.1mm")
-    (property "Sheetfile" "remote-project.kicad_sch")
+    (property "Sheetfile" "remote.kicad_sch")
     (property "Sheetname" "")
     (property "ki_description" "Generic screw terminal, single row, 01x05, script generated (kicad-library-utils/schlib/autogen/connector/)")
@@
     (pad "5" thru_hole circle (at 10.16 0 180) (size 2.1 2.1) (drill 1.1) (layers "*.Cu" "*.Mask")
       (net 1 "GND") (pinfunction "Pin_5") (pintype "passive"))
-    (model "${KICAD6_3DMODEL_DIR}/TerminalBlock_TE-Connectivity.3dshapes/TerminalBlock_TE_282834-5_1x05_P2.54mm_Horizontal.wrl"
-      (offset (xyz 0 0 0))
+    (model "/home/maximilian/.local/share/kicad/7.0/3dmodels/TE/c-282834-5-c-3d.igs"
+      (offset (xyz 5.1 -3.2 2.5))
       (scale (xyz 1 1 1))
-      (rotate (xyz 0 0 0))
+      (rotate (xyz -90 0 0))
     )
   )
   (footprint "Button_Switch:5V_LED_BTN" (layer "F.Cu")
     (at 141.675 84)
-    (property "Sheetfile" "remote-project.kicad_sch")
+    (property "Sheetfile" "remote.kicad_sch")
     (property "Sheetname" "")
     (attr through_hole)
@@
         (effects (font (size 1 1) (thickness 0.1)))
     )
-    (fp_text value "~" (at 0 1 unlocked) (layer "F.Fab")
+    (fp_text value "12mm non-resetting button" (at 0 1 unlocked) (layer "F.Fab")
         (effects (font (size 1 1) (thickness 0.15)))
     )
@@
     (descr "Mounting Hole 3.2mm, M3, DIN965")
     (tags "mounting hole 3.2mm m3 din965")
-    (property "Sheetfile" "remote-project.kicad_sch")
+    (property "Sheetfile" "remote.kicad_sch")
     (property "Sheetname" "")
     (property "ki_description" "Mounting Hole with connection")
@@
     (descr "Mounting Hole 3.2mm, M3, DIN965")
     (tags "mounting hole 3.2mm m3 din965")
-    (property "Sheetfile" "remote-project.kicad_sch")
+    (property "Sheetfile" "remote.kicad_sch")
     (property "Sheetname" "")
     (property "ki_description" "Mounting Hole with connection")
@@
     (descr "Mounting Hole 3.2mm, M3, DIN965")
     (tags "mounting hole 3.2mm m3 din965")
-    (property "Sheetfile" "remote-project.kicad_sch")
+    (property "Sheetfile" "remote.kicad_sch")
     (property "Sheetname" "")
     (property "ki_description" "Mounting Hole with connection")
@@
   (footprint "Button_Switch:5V_LED_BTN" (layer "F.Cu")
     (at 141.675 99.1)
-    (property "Sheetfile" "remote-project.kicad_sch")
+    (property "Sheetfile" "remote.kicad_sch")
     (property "Sheetname" "")
     (attr through_hole)
@@
         (effects (font (size 1 1) (thickness 0.1)))
     )
-    (fp_text value "~" (at 0 1 unlocked) (layer "F.Fab")
+    (fp_text value "12mm non-resetting button" (at 0 1 unlocked) (layer "F.Fab")
         (effects (font (size 1 1) (thickness 0.15)))
     )
@@
   (gr_line (start 126.675 49.4) (end 156.675 49.4)
     (stroke (width 0.1) (type default)) (layer "Edge.Cuts"))
+  (gr_text "JLCJLCJLCJLC" (at 135.5 51.9) (layer "F.SilkS")
+    (effects (font (size 0.7 0.7) (thickness 0.15) bold) (justify left bottom))
+  )
+  (gr_text "LightControl Remote V1.0\n03/2023 M. Stucke" (at 152.5 63.4 270) (layer "F.SilkS")
+    (effects (font (size 1.2 1.2) (thickness 0.2) bold) (justify left bottom))
+  )
   (segment (start 129.175 65.3) (end 127.8 65.3) (width 0.25) (layer "F.Cu") (net 1))
   (segment (start 129.175 95.5) (end 127.9 95.5) (width 0.25) (layer "F.Cu") (net 1))
